Commit message: Fixed typos in xacro file and remade rviz config file

File: ddr_ws/src/differential_drive_robot/urdf/differential_drive_robot.xacro.urdf (robot description, URDF)
Before this commit: robot diff_bot, 2 links, 1 joints
Joints:
- joint caster_wheel_joint: child (none) -> caster_wheel; origin xyz=${caster_wheel_offset} 0 -${caster_wheel_radius+0.05} rpy=0 0 0 -> xyz=-${caster_wheel_offset} 0 -${base_height / 2} rpy=0 0 0
